Commit message: Avidesh_branch

File: dedo/data/robots/fetch/fetch.urdf (robot description, URDF)
Before this commit: robot fetch, 26 links, 25 joints
Joints:
- joint head_pan_joint: type revolute -> fixed
- joint head_tilt_joint: type revolute -> fixed
- joint l_wheel_joint: type continuous -> fixed
- joint r_wheel_joint: type continuous -> fixed
